File: anna_elsa_credit_display/anna_elsa_credit_display.kicad_pcb (KiCad board)
At the start: 2 copper layers, 83.8 x 77.5 mm, 36 parts, among them J1 HT16K33_28, J2 I2C, J3 I2C, J4 HT16K33_20

Commit message: Latest schematics
Other:
- net class Default removed
- net class PWR removed
