File: anna_elsa_esp32_cpu/audio.kicad_sch (KiCad schematic)
At the start: 46 parts, among them J11 SPK_R, J9 SPK_L, U3 TAS5731PHP

Commit message: Latest schematics
Connections:
- net ~{RST} renamed JTAG_TMS
Other:
- note removed: "Don't connect to reset!"
Changed lines of the file:
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@@
-    (effects (font (size 1.27 1.27)) (justify left bottom))
-  )
-  (text "Don't connect to reset!" (at 182.88 124.46 0)
     (effects (font (size 1.27 1.27)) (justify left bottom))
   )
@@
   (label "PLL_FLTP" (at 52.07 148.59 0)
     (effects (font (size 1.27 1.27)) (justify left bottom))
-  )
-  (global_label "~{RST}" (shape input) (at 187.325 120.65 0) (fields_autoplaced)
-    (effects (font (size 1.27 1.27)) (justify left))
-    (property "Intersheet References" "${INTERSHEET_REFS}" (id 0) (at 193.0963 120.5706 0)
-      (effects (font (size 1.27 1.27)) (justify left) hide)
-    )
   )
   (global_label "MCLK" (shape input) (at 86.995 95.25 180) (fields_autoplaced)
@@
     )
   )
+  (global_label "JTAG_TMS" (shape input) (at 187.325 120.65 0) (fields_autoplaced)
+    (effects (font (size 1.27 1.27)) (justify left))
+    (property "Intersheet References" "${INTERSHEET_REFS}" (id 0) (at 23.495 39.37 0)
+      (effects (font (size 1.27 1.27)) hide)
+    )
+  )
