File: anna_elsa_esp32_cpu/cctalk.kicad_sch (KiCad schematic)
At the start: 11 parts, among them J7 HOPPER, J8 COIN_VALIDATOR, Q1 SS8050, Q2 SS8850

Commit message: Latest schematics
Parts:
- removed D3: BAT54, Package_TO_SOT_SMD:SOT-23, symbol anna_elsa_cpu-rescue:SCHOTTKY-w_device
- added D1: BAT54W, Package_TO_SOT_SMD:SOT-323_SC-70, symbol Diode:BAT54W
- R4, R5, R7: LCSC C25271 -> C280011
Connections:
- net CCTALK_DATA: now also D1.3 (K)
- net GND: no longer J7.2 (Pin_2), J8.2 (Pin_2)
- net HOST_RX: now also D1.1 (A); no longer Q2.3 (C), R6.1
- new net: Q2.3 (C), R6.1
- no-connect marks 10 -> 12
Other:
- moved on the sheet: R3, R6
