File: anna_elsa_moves_display/anna_elsa_moves_display.kicad_pcb (KiCad board)
At the start: 2 copper layers, 60 x 80 mm, 18 parts, among them J1 HT16K33_28, J2 I2C, J3 I2C

Commit message: Latest schematics
Other:
- net class Default removed
- net class PWR removed
