File: message_display_interface/message_display_interface.kicad_pcb (KiCad board)
At the start: 2 copper layers, 62.8 x 39.5 mm, 8 parts, among them J1 CPU, J2 VFD Display, J3 NUDGE_LED, J4 PRIZE_LED

Commit message: Added current cpu pcb and removed old
Other:
- net class Default removed
- net class PWR removed

Commit message: Latest schematics
Routing:
- net VCC: track 62.2 -> 0.00 mm
- added copper zone on F.Cu, net VCC
Changed lines of the file:
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@@
     (effects (font (size 1 1) (thickness 0.15)))
   )
-  (segment (start 153.25 82.225) (end 155.475 80) (width 0.8) (layer "F.Cu") (net 1))
-  (segment (start 152.025 65) (end 153.25 63.775) (width 0.8) (layer "F.Cu") (net 1))
-  (segment (start 155.475 80) (end 171.75 80) (width 0.8) (layer "F.Cu") (net 1))
-  (segment (start 153.25 84) (end 153.25 82.225) (width 0.8) (layer "F.Cu") (net 1))
-  (segment (start 153.25 63.775) (end 153.25 62) (width 0.8) (layer "F.Cu") (net 1))
-  (segment (start 136.54 65) (end 152.025 65) (width 0.8) (layer "F.Cu") (net 1))
-  (segment (start 153.25 62) (end 153.25 84) (width 0.8) (layer "B.Cu") (net 1))
   (segment (start 158.25 62) (end 168.75 62) (width 0.4) (layer "F.Cu") (net 6))
   (segment (start 168.75 62) (end 171.75 65) (width 0.4) (layer "F.Cu") (net 6))
@@
   (segment (start 155.75 75.25) (end 158.25 77.75) (width 0.4) (layer "B.Cu") (net 13))
   (segment (start 155.75 62) (end 155.75 75.25) (width 0.4) (layer "B.Cu") (net 13))
+  (zone (net 1) (net_name "VCC") (layer "F.Cu") (hatch edge 0.508)
+    (connect_pads (clearance 0.508))
+    (min_thickness 0.254) (filled_areas_thickness no)
+    (fill yes (thermal_gap 0.508) (thermal_bridge_width 0.508))
+    (polygon
+      (pts
+        (xy 182.5 93)
+        (xy 119.75 93)
+        (xy 119.75 53.5)
+        (xy 182.5 53.5)
+      )
+    )
+  )
   (zone (net 5) (net_name "GND") (layer "B.Cu") (hatch edge 0.508)
     (connect_pads (clearance 0.508))
-    (min_thickness 0.254)
+    (min_thickness 0.254) (filled_areas_thickness no)
     (fill yes (thermal_gap 0.508) (thermal_bridge_width 0.508))
     (polygon
